File: Arduino-Mini-Drone-KiCad/Arduino-Mini-Drone-KiCad.kicad_sch (KiCad schematic)
At the start: 74 parts, among them J1 NRF24, J10 BT, J11 PPM, J12 PWR, J13 Open, J2 UART, J3 Motor1, J4 Motor2, J5 Motor3, J6 Motor4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

Commit message: added mpu9250 lib & completed PCB layout
Parts:
- added H1, H2: MountingHole, MountingHole:MountingHole_2.2mm_M2_Pad_Via, symbol Mechanical:MountingHole
- BZ1, JP2, JP3: footprint (none) -> Connector_PinHeader_2.54mm:PinHeader_1x02_P2.54mm_Vertical
- C1, C2, C3, C6: footprint (none) -> Capacitor_SMD:C_0402_1005Metric; LCSC (none) -> C71629
- C10, C11, C12, C13: footprint (none) -> Capacitor_SMD:C_0603_1608Metric; LCSC (none) -> C109447
- C14, C15: footprint (none) -> Capacitor_Tantalum_SMD:CP_EIA-6032-15_Kemet-U; LCSC (none) -> C171664
- C16: footprint (none) -> Capacitor_SMD:C_0603_1608Metric; symbol Device:C_Polarized_US -> Device:C; LCSC (none) -> C14663
- C17: footprint (none) -> Capacitor_SMD:C_0603_1608Metric; LCSC (none) -> C380316
- C18, C19, C20, C21, C22: footprint (none) -> Capacitor_SMD:C_0603_1608Metric; LCSC (none) -> C14663
- C4, C5, C9: footprint (none) -> Capacitor_Tantalum_SMD:CP_EIA-6032-15_Kemet-U; LCSC (none) -> C600516
- C7, C8: footprint (none) -> Capacitor_SMD:C_0603_1608Metric; LCSC (none) -> C15849
- D1: footprint (none) -> LED_SMD:LED_0603_1608Metric; LCSC (none) -> C241891
- D10, D7, D8, D9: LCSC (none) -> C2761795
- D2: footprint (none) -> LED_SMD:LED_0603_1608Metric; LCSC (none) -> C266784
- D3, D4, D5, D6: LCSC (none) -> C3011102
- J1: footprint (none) -> Connector_PinHeader_1.27mm:PinHeader_1x08_P1.27mm_Vertical
- J10: footprint (none) -> Connector_PinSocket_2.54mm:PinSocket_1x04_P2.54mm_Vertical
- J11: footprint (none) -> Connector_PinSocket_2.54mm:PinSocket_1x03_P2.54mm_Vertical
- J12, J3, J4, J5, J6: footprint (none) -> Connector_JST:JST_PH_B2B-PH-K_1x02_P2.00mm_Vertical
- J13, J2: footprint (none) -> Connector_PinHeader_2.54mm:PinHeader_1x05_P2.54mm_Vertical
- J7: value Conn_01x02 -> CapHole; footprint (none) -> Connector_PinSocket_2.54mm:PinSocket_1x02_P2.54mm_Vertical
- J8: footprint (none) -> Connector_PinSocket_2.54mm:PinSocket_1x08_P2.54mm_Vertical
- J9: footprint (none) -> Connector_PinHeader_2.54mm:PinHeader_1x04_P2.54mm_Vertical
- JP1: footprint (none) -> Jumper:SolderJumper-2_P1.3mm_Open_Pad1.0x1.5mm
- Q1, Q2, Q3, Q4: LCSC (none) -> C347475
- Q5: LCSC (none) -> C347476
- R1, R10, R3, R4, R6, R8: footprint (none) -> Resistor_SMD:R_0603_1608Metric; LCSC (none) -> C25804
- R11, R5, R7, R9: footprint (none) -> Resistor_SMD:R_0603_1608Metric; LCSC (none) -> C19702
- R12: footprint (none) -> Resistor_SMD:R_0603_1608Metric; LCSC (none) -> C25803
- R13: footprint (none) -> Resistor_SMD:R_0603_1608Metric; LCSC (none) -> C4216
- R14: footprint (none) -> Resistor_SMD:R_0603_1608Metric; LCSC (none) -> C23151
- R2: footprint (none) -> Resistor_SMD:R_0603_1608Metric; LCSC (none) -> C23140
- SW1: footprint (none) -> Button_Switch_SMD:SW_Tactile_SPST_NO_Straight_CK_PTS636Sx25SMTRLFS; LCSC (none) -> C483881
- SW2: footprint (none) -> Button_Switch_THT:SW_CuK_OS102011MA1QN1_SPDT_Angled
- U1: LCSC (none) -> C14877
- U2: LCSC (none) -> C412820
- U3: LCSC (none) -> C5370990
- Y1: footprint (none) -> Crystal:Crystal_SMD_3225-4Pin_3.2x2.5mm; symbol Device:Crystal_GND2 -> Device:Crystal_GND23_Small; LCSC (none) -> C124318
Connections:
- net +BATT: no longer C19.2, C20.2, C21.2, C22.2, D10.1 (VDD), D7.1 (VDD), D8.1 (VDD), D9.1 (VDD)
- net A1: now also J13.3 (Pin_3); no longer J13.1 (Pin_1)
- net A2: now also J13.4 (Pin_4); no longer J13.2 (Pin_2)
- net A3: now also J13.5 (Pin_5); no longer J13.3 (Pin_3)
- net A6: now also J13.1 (Pin_1); no longer J13.4 (Pin_4)
- net A7: now also J13.2 (Pin_2); no longer J13.5 (Pin_5)
- net D3: now also R6.2, R7.2; no longer R10.2, R11.2
- net D5: now also R4.2, R5.2; no longer R8.2, R9.2
- net D6: now also R8.2, R9.2; no longer R6.2, R7.2
- net D9: now also R10.2, R11.2; no longer R4.2, R5.2
- net GND: now also Y1.3
- net VMOT: now also C19.2, C20.2, C21.2, C22.2, D10.1 (VDD), D7.1 (VDD), D8.1 (VDD), D9.1 (VDD)
- net at D10.2 (DOUT): now also D7.4 (DIN)
- net at U1.7 (XTAL1/PB6): now also Y1.4; no longer Y1.3
- net at R14.2: now also D9.4 (DIN); no longer D7.4 (DIN)
- net at D8.2 (DOUT): no longer D9.4 (DIN)
Other:
- moved on the sheet: D7, D8, D9, Y1
