File: Arduino-Mini-Drone-KiCad/V2/Arduino-Mini-Drone-KiCad.kicad_pcb (KiCad board)
At the start: 2 copper layers, 58.8 x 59.1 mm, 79 parts, among them J1 NRF24, J10 BT, J11 PPM, J12 PWR, J13 Open, J2 UART, J3 Motor1, J4 Motor2, J5 Motor3, J6 Motor4, J7 CapHole, J8 MPU9250 + BMP280, J9 SPI Pads, Q1 AO3400A, Q2 AO3400A, Q3 AO3400A, Q4 AO3400A, Q5 AO3401A, SW1 Reset, SW2 Switch, U1 ATmega328P-A, U2 MIC5205YM5, U3 LP5907MFX-3.3, Y1 Crystal_GND2

Commit message: Completed Panelized PCB in V2 delete Row 2 PCB for error resolution
Parts:
- removed ?: LOGO, LOGO
- removed J10: BT, Connector_PinSocket_2.54mm:PinSocket_1x04_P2.54mm_Vertical
- removed J5: Motor3, Connector_JST:JST_PH_B2B-PH-K_1x02_P2.00mm_Vertical
- removed J6: Motor4, Connector_JST:JST_PH_B2B-PH-K_1x02_P2.00mm_Vertical
- removed J9: SPI Pads, Connector_PinHeader_2.54mm:PinHeader_1x04_P2.54mm_Vertical
- removed JP1: Power isolation jumper (low power applications), Jumper:SolderJumper-2_P1.3mm_Open_Pad1.0x1.5mm
- removed JP2, JP3: Power isolation jumper (low power applications), Connector_PinHeader_2.54mm:PinHeader_1x02_P2.54mm_Vertical
- removed SW1: Reset, Button_Switch_SMD:SW_Tactile_SPST_NO_Straight_CK_PTS636Sx25SMTRLFS
- removed SW2: Switch, Button_Switch_THT:SW_CuK_OS102011MA1QN1_SPDT_Angled
- added B+: PWR, Connector_JST:JST_PH_B2B-PH-K_1x02_P2.00mm_Vertical, F.Cu at (228.8, 36.8)
- added B+1: PWR, Connector_JST:JST_PH_B2B-PH-K_1x02_P2.00mm_Vertical, F.Cu at (237.6, 83.7)
- added BZ2: Buzzer, Connector_PinHeader_1.27mm:PinHeader_1x02_P1.27mm_Vertical, F.Cu at (230.9, 87.1)
- added C25: 1uf, Capacitor_SMD:C_0603_1608Metric_Pad1.08x0.95mm_HandSolder, F.Cu at (201.3, 74.1)
- added C26: 1uf, Capacitor_SMD:C_0603_1608Metric_Pad1.08x0.95mm_HandSolder, F.Cu at (201.3, 81.3)
- added C27: 10uf, Capacitor_SMD:C_1206_3216Metric_Pad1.33x1.80mm_HandSolder, F.Cu at (208.7, 96.1)
- added C28: 22uf, Capacitor_SMD:C_0805_2012Metric_Pad1.18x1.45mm_HandSolder, F.Cu at (256.9, 71.5)
- added C29: 22uf, Capacitor_SMD:C_0805_2012Metric_Pad1.18x1.45mm_HandSolder, F.Cu at (258.4, 94.5)
- added C30: 22uf, Capacitor_SMD:C_0805_2012Metric_Pad1.18x1.45mm_HandSolder, F.Cu at (258.2, 81.2)
- added C31: 22uf, Capacitor_SMD:C_0805_2012Metric_Pad1.18x1.45mm_HandSolder, F.Cu at (247.5, 71.7)
- added C32: 100uf, Capacitor_Tantalum_SMD:CP_EIA-3528-12_Kemet-T_Pad1.50x2.35mm_HandSolder, F.Cu at (241.9, 85.5)
- added C33: 100uf, Capacitor_Tantalum_SMD:CP_EIA-3528-12_Kemet-T_Pad1.50x2.35mm_HandSolder, F.Cu at (237.2, 79.0)
- added C34: 10uf, Capacitor_SMD:C_0603_1608Metric_Pad1.08x0.95mm_HandSolder, F.Cu at (246.5, 91.3)
- added C35: 100nf, Capacitor_SMD:C_0603_1608Metric_Pad1.08x0.95mm_HandSolder, F.Cu at (246.6, 95.0)
- added C36: 100nf, Capacitor_SMD:C_0603_1608Metric_Pad1.08x0.95mm_HandSolder, B.Cu at (256.9, 91.7)
- added D11: SS34, Diode_SMD:D_MELF_Handsoldering, F.Cu at (258.3, 90.1)
- added D12: SS34, Diode_SMD:D_MELF_Handsoldering, F.Cu at (258.5, 85.2)
- added D13: SS34, Diode_SMD:D_MELF_Handsoldering, F.Cu at (251.6, 71.6)
- added D14: WS2812B, LED_SMD:LED_WS2812B_PLCC4_5.0x5.0mm_P3.2mm, B.Cu at (259.6, 96.5)
- added G***: LOGO, LOGO, F.Cu at (243.6, 48.7)
- added G***: LOGO, LOGO, B.Cu at (244.0, 48.4)
- added G***1: LOGO, LOGO, F.Cu at (222.8, 71.7)
- added G***2: LOGO, LOGO, B.Cu at (222.4, 72.1)
- added H10: MountingHole, MountingHole:MountingHole_2.2mm_M2_Pad_Via, F.Cu at (225.3, 93.7)
- added H11: MountingHole, MountingHole:MountingHole_2.2mm_M2_Pad_Via, F.Cu at (225.3, 68.2)
- added H12: MountingHole, MountingHole:MountingHole_2.2mm_M2_Pad_Via, F.Cu at (199.8, 68.2)
- added H13: MountingHole, MountingHole:MountingHole_2.2mm_M2_Pad_Via, F.Cu at (266.8, 93.7)
- added H14: MountingHole, MountingHole:MountingHole_2.2mm_M2_Pad_Via, F.Cu at (266.9, 68.2)
- added H15: MountingHole, MountingHole:MountingHole_2.2mm_M2_Pad_Via, F.Cu at (241.3, 68.2)
- added H16: MountingHole, MountingHole:MountingHole_2.2mm_M2_Pad_Via, F.Cu at (241.3, 93.7)
- added H3: MountingHole, MountingHole:MountingHole_2.2mm_M2_Pad_Via, F.Cu at (241.2, 52.3)
- added H4: MountingHole, MountingHole:MountingHole_2.2mm_M2_Pad_Via, F.Cu at (266.7, 52.3)
- added H5: MountingHole, MountingHole:MountingHole_2.2mm_M2_Pad_Via, F.Cu at (199.6, 26.7)
- added H6: MountingHole, MountingHole:MountingHole_2.2mm_M2_Pad_Via, F.Cu at (199.6, 52.2)
- added H7: MountingHole, MountingHole:MountingHole_2.2mm_M2_Pad_Via, F.Cu at (225.1, 52.2)
- added H8: MountingHole, MountingHole:MountingHole_2.2mm_M2_Pad_Via, F.Cu at (225.1, 26.7)
- added H9: MountingHole, MountingHole:MountingHole_2.2mm_M2_Pad_Via, F.Cu at (199.8, 93.7)
- added J14: Open, Connector_PinHeader_1.27mm:PinHeader_1x05_P1.27mm_Vertical, F.Cu at (230.9, 83.4)
- added M1: Motor1, Connector_PinHeader_1.27mm:PinHeader_1x02_P1.27mm_Vertical, F.Cu at (211.1, 57.8)
- added M2: Motor2, Connector_PinHeader_1.27mm:PinHeader_1x02_P1.27mm_Vertical, F.Cu at (194.1, 38.2)
- added M3: Motor3, Connector_PinHeader_1.27mm:PinHeader_1x02_P1.27mm_Vertical, F.Cu at (194.1, 40.8)
- added M4: Motor4, Connector_PinHeader_1.27mm:PinHeader_1x02_P1.27mm_Vertical, F.Cu at (213.7, 57.8)
- added M5: Motor1, Connector_PinHeader_1.27mm:PinHeader_1x02_P1.27mm_Vertical, F.Cu at (255.4, 62.6)
- added M6: Motor2, Connector_PinHeader_1.27mm:PinHeader_1x02_P1.27mm_Vertical, F.Cu at (272.4, 82.3)
- added M7: Motor3, Connector_PinHeader_1.27mm:PinHeader_1x02_P1.27mm_Vertical, F.Cu at (272.4, 79.6)
- added M8: Motor4, Connector_PinHeader_1.27mm:PinHeader_1x02_P1.27mm_Vertical, F.Cu at (252.8, 62.6)
- added NEO: POWER, Connector_PinHeader_1.27mm:PinHeader_1x08_P1.27mm_Vertical, F.Cu at (221.1, 21.2)
- added NEO1: POWER, Connector_PinHeader_1.27mm:PinHeader_1x08_P1.27mm_Vertical, F.Cu at (245.4, 99.2)
- added NEO_Enable: LED ON OFF, Jumper:SolderJumper-2_P1.3mm_Open_Pad1.0x1.5mm, B.Cu at (205.8, 29.3)
- added NEO_Enable1: LED ON OFF, Jumper:SolderJumper-2_P1.3mm_Open_Pad1.0x1.5mm, B.Cu at (260.7, 91.2)
- added Q10: AO3401A, Package_TO_SOT_SMD:SOT-23, F.Cu at (242.2, 80.8)
- added Q6: AO3400A, Package_TO_SOT_SMD:SOT-23, F.Cu at (256.9, 68.0)
- added Q7: AO3400A, Package_TO_SOT_SMD:SOT-23, F.Cu at (254.6, 94.5)
- added Q8: AO3400A, Package_TO_SOT_SMD:SOT-23, F.Cu at (262.2, 81.2)
- added Q9: AO3400A, Package_TO_SOT_SMD:SOT-23, F.Cu at (247.4, 68.0)
- added R15: 10K, Resistor_SMD:R_0603_1608Metric_Pad0.98x0.95mm_HandSolder, F.Cu at (213.8, 77.7)
- added R16: 330, Resistor_SMD:R_0603_1608Metric_Pad0.98x0.95mm_HandSolder, F.Cu at (224.3, 88.7)
- added R17: 10k, Resistor_SMD:R_0603_1608Metric_Pad0.98x0.95mm_HandSolder, F.Cu at (206.1, 77.2)
- added R18: 10k, Resistor_SMD:R_0603_1608Metric_Pad0.98x0.95mm_HandSolder, F.Cu at (258.0, 75.3)
- added R19: 100, Resistor_SMD:R_0603_1608Metric_Pad0.98x0.95mm_HandSolder, F.Cu at (255.7, 75.3)
- added R20: 10k, Resistor_SMD:R_0603_1608Metric_Pad0.98x0.95mm_HandSolder, F.Cu at (262.0, 93.3)
- added R21: 100, Resistor_SMD:R_0603_1608Metric_Pad0.98x0.95mm_HandSolder, F.Cu at (262.0, 95.6)
- added R22: 10k, Resistor_SMD:R_0603_1608Metric_Pad0.98x0.95mm_HandSolder, F.Cu at (254.8, 82.1)
- added R23: 100, Resistor_SMD:R_0603_1608Metric_Pad0.98x0.95mm_HandSolder, F.Cu at (254.8, 80.0)
- added R24: 10k, Resistor_SMD:R_0603_1608Metric_Pad0.98x0.95mm_HandSolder, F.Cu at (248.6, 75.4)
- added R25: 100, Resistor_SMD:R_0603_1608Metric_Pad0.98x0.95mm_HandSolder, F.Cu at (246.6, 75.4)
- added R26: 100k, Resistor_SMD:R_0603_1608Metric_Pad0.98x0.95mm_HandSolder, F.Cu at (246.6, 89.3)
- added R27: 33k, Resistor_SMD:R_0603_1608Metric_Pad0.98x0.95mm_HandSolder, F.Cu at (246.5, 93.2)
- added R28: 390, Resistor_SMD:R_0603_1608Metric_Pad0.98x0.95mm_HandSolder, B.Cu at (255.4, 94.8)
- added U4: ATmega328P-A, Package_QFP:TQFP-32_7x7mm_P0.8mm, F.Cu at (214.9, 88.2)
- added U5: MIC5205YM5, Package_TO_SOT_SMD:SOT-23-5_HandSoldering, F.Cu at (206.2, 73.3)
- added U6: LP5907MFX-3.3, Package_TO_SOT_SMD:SOT-23-5_HandSoldering, F.Cu at (201.3, 77.7)
- added VCC: MPU9250 + BMP280, Connector_PinSocket_2.54mm:PinSocket_1x05_P2.54mm_Vertical, F.Cu at (243.6, 42.7)
- added VCC1: MPU9250 + BMP280, Connector_PinSocket_2.54mm:PinSocket_1x05_P2.54mm_Vertical, F.Cu at (222.9, 77.7)
- added Y2: Crystal_GND2, Crystal:Crystal_SMD_5032-4Pin_5.0x3.2mm, F.Cu at (201.6, 85.5)
- added mouse-bite-2mm-slot: VAL**, Panelization.pretty-master:mouse-bite-2mm-slot, F.Cu at (233.2, 29.8)
- added mouse-bite-2mm-slot: VAL**, Panelization.pretty-master:mouse-bite-2mm-slot, F.Cu at (233.2, 47.7)
- added mouse-bite-2mm-slot1: VAL**, Panelization.pretty-master:mouse-bite-2mm-slot, F.Cu at (262.8, 60.2)
- added mouse-bite-2mm-slot1: VAL**, Panelization.pretty-master:mouse-bite-2mm-slot, F.Cu at (233.3, 72.8)
- added mouse-bite-2mm-slot1: VAL**, Panelization.pretty-master:mouse-bite-2mm-slot, F.Cu at (203.3, 60.2)
- added mouse-bite-2mm-slot1: VAL**, Panelization.pretty-master:mouse-bite-2mm-slot, F.Cu at (220.4, 60.2)
- added mouse-bite-2mm-slot1: VAL**, Panelization.pretty-master:mouse-bite-2mm-slot, F.Cu at (233.3, 90.8)
- added mouse-bite-2mm-slot1: VAL**, Panelization.pretty-master:mouse-bite-2mm-slot, F.Cu at (245.9, 60.2)
- BZ1: footprint Connector_PinHeader_2.54mm:PinHeader_1x02_P2.54mm_Vertical -> Connector_PinHeader_1.27mm:PinHeader_1x02_P1.27mm_Vertical
- C1, C2, C3, C6: footprint Capacitor_SMD:C_0402_1005Metric -> Capacitor_SMD:C_0603_1608Metric_Pad1.08x0.95mm_HandSolder
- C10, C11, C12, C13: footprint Capacitor_SMD:C_0603_1608Metric -> Capacitor_SMD:C_0805_2012Metric_Pad1.18x1.45mm_HandSolder
- C14, C15: footprint Capacitor_Tantalum_SMD:CP_EIA-6032-15_Kemet-U -> Capacitor_Tantalum_SMD:CP_EIA-3528-12_Kemet-T_Pad1.50x2.35mm_HandSolder
- C16, C20, C21: value 100nf -> 0.1uf; footprint Capacitor_SMD:C_0603_1608Metric -> Capacitor_SMD:C_0603_1608Metric_Pad1.08x0.95mm_HandSolder
- C17, C18, C7, C8: footprint Capacitor_SMD:C_0603_1608Metric -> Capacitor_SMD:C_0603_1608Metric_Pad1.08x0.95mm_HandSolder
- C19: footprint Capacitor_SMD:C_0603_1608Metric -> Capacitor_SMD:C_0603_1608Metric_Pad1.08x0.95mm_HandSolder; moved to B.Cu
- C22: value 100nf -> 10uf; footprint Capacitor_SMD:C_0603_1608Metric -> Capacitor_Tantalum_SMD:CP_EIA-3216-10_Kemet-I_Pad1.58x1.35mm_HandSolder
- C23: value 0.1uf -> 10uf; footprint Capacitor_SMD:C_0805_2012Metric -> Capacitor_Tantalum_SMD:CP_EIA-3216-10_Kemet-I_Pad1.58x1.35mm_HandSolder
- C24: footprint Capacitor_SMD:C_0805_2012Metric -> Capacitor_SMD:C_0603_1608Metric_Pad1.08x0.95mm_HandSolder
- C4, C5: footprint Capacitor_Tantalum_SMD:CP_EIA-6032-15_Kemet-U -> Capacitor_Tantalum_SMD:CP_EIA-3216-10_Kemet-I_Pad1.58x1.35mm_HandSolder
- C9: footprint Capacitor_Tantalum_SMD:CP_EIA-6032-15_Kemet-U -> Capacitor_SMD:C_1206_3216Metric_Pad1.33x1.80mm_HandSolder
- D1, D2: footprint LED_SMD:LED_0603_1608Metric -> LED_SMD:LED_0603_1608Metric_Pad1.05x0.95mm_HandSolder
- D10: value WS2812B -> SS34; footprint LED_SMD:LED_WS2812B_PLCC4_5.0x5.0mm_P3.2mm -> Diode_SMD:D_MELF_Handsoldering
- D3, D4, D5, D6: footprint Diode_SMD:D_MELF -> Diode_SMD:D_MELF_Handsoldering
- D7: value WS2812B -> Green; footprint LED_SMD:LED_WS2812B_PLCC4_5.0x5.0mm_P3.2mm -> LED_SMD:LED_0603_1608Metric_Pad1.05x0.95mm_HandSolder
- D8: value WS2812B -> Red; footprint LED_SMD:LED_WS2812B_PLCC4_5.0x5.0mm_P3.2mm -> LED_SMD:LED_0603_1608Metric_Pad1.05x0.95mm_HandSolder
- D9: moved to B.Cu
- J11: footprint Connector_PinSocket_2.54mm:PinSocket_1x03_P2.54mm_Vertical -> Connector_PinHeader_1.27mm:PinHeader_1x03_P1.27mm_Vertical
- J12: value PWR -> PPM; footprint Connector_JST:JST_PH_B2B-PH-K_1x02_P2.00mm_Vertical -> Connector_PinHeader_1.27mm:PinHeader_1x03_P1.27mm_Vertical
- J13: footprint Connector_PinHeader_2.54mm:PinHeader_1x05_P2.54mm_Vertical -> Connector_PinHeader_1.27mm:PinHeader_1x05_P1.27mm_Vertical
- J2: value UART -> UART + BT; footprint Connector_PinHeader_2.54mm:PinHeader_1x05_P2.54mm_Vertical -> Connector_PinHeader_1.27mm:PinHeader_1x06_P1.27mm_Vertical
- J3: value Motor1 -> NRF24; footprint Connector_JST:JST_PH_B2B-PH-K_1x02_P2.00mm_Vertical -> Connector_PinHeader_1.27mm:PinHeader_1x08_P1.27mm_Vertical
- J4: value Motor2 -> UART + BT; footprint Connector_JST:JST_PH_B2B-PH-K_1x02_P2.00mm_Vertical -> Connector_PinHeader_1.27mm:PinHeader_1x06_P1.27mm_Vertical
- J7: value CapHole -> MCU; footprint Connector_PinSocket_2.54mm:PinSocket_1x02_P2.54mm_Vertical -> Connector_PinHeader_1.27mm:PinHeader_1x08_P1.27mm_Vertical
- J8: value MPU9250 + BMP280 -> MCU; footprint Connector_PinSocket_2.54mm:PinSocket_1x08_P2.54mm_Vertical -> Connector_PinHeader_1.27mm:PinHeader_1x08_P1.27mm_Vertical
- R1, R10, R11, R12, R13, R2, R3, R4, R5, R6, R7, R8, R9: footprint Resistor_SMD:R_0603_1608Metric -> Resistor_SMD:R_0603_1608Metric_Pad0.98x0.95mm_HandSolder
- R14: footprint Resistor_SMD:R_0603_1608Metric -> Resistor_SMD:R_0603_1608Metric_Pad0.98x0.95mm_HandSolder; moved to B.Cu
- U2, U3: footprint Package_TO_SOT_SMD:SOT-23-5 -> Package_TO_SOT_SMD:SOT-23-5_HandSoldering
- Y1: footprint Crystal:Crystal_SMD_3225-4Pin_3.2x2.5mm -> Crystal:Crystal_SMD_5032-4Pin_5.0x3.2mm
- moved C6 194.4 mm to (259.6, 38.0), turned to 0 degrees
- moved C8 193.8 mm to (265.2, 39.1), turned to 180 degrees
- moved H2 192.5 mm to (241.2, 26.8), turned to -90 degrees
- moved U3 191.8 mm to (265.2, 42.7), turned to 90 degrees
- moved C7 190.4 mm to (265.2, 46.4), turned to 0 degrees
- moved R3 190.0 mm to (260.4, 43.2)
- moved J7 187.5 mm to (272.3, 33.4), turned to 0 degrees
- moved C4 186.4 mm to (260.4, 51.1), turned to 180 degrees
- moved C9 186.3 mm to (257.8, 24.3), turned to 0 degrees
- moved D2 186.0 mm to (257.1, 43.9), turned to 90 degrees
- moved U2 183.9 mm to (260.3, 47.2)
- moved Y1 182.3 mm to (264.9, 34.9), turned to 0 degrees
- moved J1 181.6 mm to (247.1, 21.2), turned to 90 degrees
- moved C5 181.3 mm to (258.8, 40.5), turned to 0 degrees
- moved D10 177.5 mm to (261.2, 71.5), turned to 90 degrees
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Connections:
- BZ1 pad 1: D8 -> D2
- BZ1 pad 2: GND -> -BATT
- C10 pad 1: GND -> -BATT
- C11 pad 1: GND -> -BATT
- C12 pad 1: GND -> -BATT
- C13 pad 1: GND -> -BATT
- C14 pad 1: RAW -> +BATT
- C14 pad 2: GND -> -BATT
- C15 pad 1: RAW -> +BATT
- C15 pad 2: GND -> -BATT
- C16 pad 1: RAW -> RST
- C16 pad 2: GND -> DTR
- C17 pad 1: GND -> -BATT
- C17 pad 2: RAW -> +BATT
- C18 pad 1: GND -> -BATT
- C18 pad 2: A0 -> BATT LVL
- C19 pad 1: GND -> -BATT
- C19 pad 2: VMOT -> +BATT
- C2 pad 1: GND -> -BATT
- C20 pad 1: GND -> -BATT
- C20 pad 2: VMOT -> Net-(U1-AREF)
- C21 pad 1: GND -> -BATT
- C21 pad 2: VMOT -> VCC
- C22 pad 1: GND -> +BATT IN
- C22 pad 2: VMOT -> -BATT
- C23 pad 1: GND -> VCC
- C23 pad 2: Net-(U1-XTAL1/PB6) -> -BATT
- C24 pad 1: GND -> -BATT
- C24 pad 2: Net-(U1-XTAL2/PB7) -> VCC
- C3 pad 1: GND -> -BATT
- C4 pad 1: RAW -> +BATT IN
- C4 pad 2: GND -> -BATT
- C5 pad 2: GND -> -BATT
- C6 pad 1: GND -> -BATT
- C7 pad 1: GND -> -BATT
- C7 pad 2: RAW -> +BATT IN
- C8 pad 1: GND -> -BATT
- C9 pad 2: GND -> -BATT
- D1 pad 1: GND -> -BATT
- D10 pad 2: Net-(D10-DOUT) -> Net-(D3-A)
- D2 pad 2: Net-(D2-A) -> VCC
- D7 pad 1: VMOT -> -BATT
- D7 pad 2: Net-(D7-DOUT) -> Net-(D1-A)
- D8 pad 1: VMOT -> Net-(D2-K)
- D8 pad 2: unconnected-(D8-DOUT-Pad2) -> VCC
- D9 pad 1: VMOT -> +BATT
- D9 pad 2: Net-(D10-DIN) -> unconnected-(D9-DOUT-Pad2)
- D9 pad 3: Net-(D10-VSS) -> Net-(D9-VSS)
- H1 pad 1: (no net) -> -BATT
- H2 pad 1: (no net) -> -BATT
- J1 pad 7: GND -> -BATT
- J11 pad 1: GND -> -BATT
- J11 pad 3: D2 -> D8
- J12 pad 2: RAW -> VCC
- J13 pad 3: A1 -> A0
- J13 pad 4: A2 -> A1
- J13 pad 5: A3 -> A2
- J2 pad 3: GND -> -BATT
- J3 pad 1: VMOT -> unconnected-(J1-Pin_1-Pad1)
- J3 pad 2: Net-(D3-A) -> D12
- J4 pad 1: VMOT -> DTR
- J4 pad 2: Net-(D4-A) -> VCC
- J7 pad 1: GND -> D6
- J7 pad 2: VMOT -> D5
- J8 pad 1: unconnected-(J8-Pin_1-Pad1) -> D6
- J8 pad 2: unconnected-(J8-Pin_2-Pad2) -> D5
- J8 pad 3: unconnected-(J8-Pin_3-Pad3) -> D9
- J8 pad 4: A4 -> D4
- J8 pad 5: A5 -> D3
- J8 pad 6: GND -> A3
- J8 pad 7: unconnected-(J8-Pin_7-Pad7) -> +BATT IN
- J8 pad 8: RAW -> -BATT
- Q1 pad 2: GND -> -BATT
- Q2 pad 2: GND -> -BATT
- Q3 pad 2: GND -> -BATT
- Q4 pad 2: GND -> -BATT
- Q5 pad 1: GND -> -BATT
- Q5 pad 2: RAW -> +BATT
- Q5 pad 3: Net-(JP3-B) -> VMOT
- R10 pad 1: GND -> -BATT
- R10 pad 2: D9 -> M4
- R11 pad 2: D9 -> M4
- R12 pad 1: RAW -> +BATT
- R12 pad 2: A0 -> BATT LVL
- R13 pad 1: A0 -> BATT LVL
- R13 pad 2: GND -> -BATT
- R14 pad 1: D4 -> D4 IN
- R3 pad 1: GND -> -BATT
- R4 pad 1: GND -> -BATT
- R4 pad 2: D5 -> M1
- R5 pad 2: D5 -> M1
- R6 pad 1: GND -> -BATT
- R6 pad 2: D3 -> M2
- R7 pad 2: D3 -> M2
- R8 pad 1: GND -> -BATT
- R8 pad 2: D6 -> M3
- R9 pad 2: D6 -> M3
- U1 pad 21: GND -> -BATT
- U1 pad 3: GND -> -BATT
- U1 pad 5: GND -> -BATT
- U2 pad 1: RAW -> +BATT IN
- U2 pad 2: GND -> -BATT
- U2 pad 3: RAW -> +BATT IN
- U2 pad 5: Net-(D2-A) -> VCC
- U3 pad 1: RAW -> +BATT IN
- U3 pad 2: GND -> -BATT
- U3 pad 3: RAW -> +BATT IN
- Y1 pad 1: Net-(U1-XTAL2/PB7) -> Net-(U1-XTAL1/PB6)
- Y1 pad 2: GND -> -BATT
- Y1 pad 3: GND -> -BATT
- Y1 pad 4: Net-(U1-XTAL1/PB6) -> Net-(U1-XTAL2/PB7)
Routing:
- net -BATT: track 13.3 -> 274.8 mm, vias 0 -> 18
- net Net-(D10-VSS): track 140.4 -> 0.00 mm, vias 2 -> 0
- net +BATT: track 0.00 -> 134.5 mm
- net RAW: track 133.4 -> 0.00 mm, vias 3 -> 0
- net VCC: track 91.7 -> 198.2 mm, vias 4 -> 2
- net Net-(D10-DOUT): track 73.9 -> 0.00 mm, vias 2 -> 0
- net Net-(D7-DOUT): track 65.1 -> 0.00 mm
- net M1: track 0.00 -> 55.0 mm
- net +BATT IN: track 0.00 -> 53.7 mm
- net M4: track 0.00 -> 50.9 mm
- net +3.3V: track 16.2 -> 61.5 mm, vias 0 -> 4
- net A3: track 12.8 -> 54.8 mm, vias 0 -> 2
- net M3: track 0.00 -> 40.7 mm
- net Net-(D10-DIN): track 40.1 -> 0.00 mm, vias 2 -> 0
- net Net-(D4-A): track 9.83 -> 47.6 mm
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- added copper zone on B.Cu, net -BATT
- added copper zone on F.Cu, net -BATT
- removed copper zone on B.Cu, net GND
- removed copper zone on F.Cu, net GND
Other:
- board size 58.8 x 59.1 mm -> 81.7 x 81.5 mm
- board text added: "- D2"
- board text added: "6 7 0 1 2"
- board text added: "B+"
- board text added: "B-"
- board text added: "BAT-"
- board text added: "BATT_LVL"
- board text added: "D11/MOSI"
- board text added: "D12/MISO"
- board text added: "D13/SCK"
- board text added: "D8"
- board text added: "DTR"
- board text added: "Gaurav B"
- board text added: "L M1 M2 M3 M4 B +-"
- board text added: "RST"
- board text added: "RX1"
- board text added: "TX0"
- board text added: "V0 by"
- board text added: "VCC"
- board text added: "VCC -"
- board text removed: "+"
- board text removed: "A3 A2 A7 A7 A6"
- board text removed: "A6 A7 A1 A2 A3"
- board text removed: "Arduino Mini Drone V1"
- board text removed: "BATTERY"
- board text removed: "BT"
- board text removed: "CAP"
- board text removed: "D2 VCC GND"
- board text removed: "DTR VCC GND RX TX"
- board text removed: "GND VCC D2"
- board text removed: "LED ON/OFF"
- board text removed: "MISO MOSI SCK RST"
- board text removed: "MOTORS ON/OFF"
- board text removed: "MPU"
- board text removed: "OFF ON"
- board text removed: "ON OFF"
- board text removed: "PPM"
- board text removed: "SPI"
- board text removed: "TX RX GND VCC"
- board text removed: "TX RX GND VCC DTR"
- board text removed: "UART"
- board text removed: "VCC GND A5 A4"
- board text removed: "VCC GND RX TX"
